Commit message: ".gitignore"

File: vslam_dev_ws/install/camera_gazebo/share/camera_gazebo/description/bu.xacro (robot description, xacro)
@@ -1,166 +1 @@
-<?xml version="1.0"?>
-<robot xmlns:xacro="http://www.ros.org/wiki/xacro" name="camera_robot">
-    <material name="white">
-        <color rgba="1 1 1 1"/>
-    </material>
-    <material name="orange">
-        <color rgba="1 0.3 0.1 1"/>
-    </material>
-    <material name="blue">
-        <color rgba="0.2 0.2 1 1"/>
-    </material>
-    <gazebo reference="base_link">
-        <material>Gazebo/Green</material>
-        <!-- <gravity>0</gravity> -->
-    </gazebo>
-    <gazebo reference="slider_link">
-        <material>Gazebo/Blue</material>
-        <!-- <gravity>0</gravity> -->
-    </gazebo>
-    <xacro:macro name="inertial_sphere" params="mass radius *origin">
-        <inertial>
-            <xacro:insert_block name="origin"/>
-            <mass value="${mass}" />
-            <inertia ixx="${(2/5) * mass * (radius*radius)}" ixy="0.0" ixz="0.0"
-                    iyy="${(2/5) * mass * (radius*radius)}" iyz="0.0"
-                    izz="${(2/5) * mass * (radius*radius)}" />
-        </inertial>
-    </xacro:macro>
-    <xacro:macro name="inertial_box" params="mass x y z *origin">
-        <inertial>
-            <xacro:insert_block name="origin"/>
-            <mass value="${mass}" />
-            <inertia ixx="${(1/12) * mass * (y*y+z*z)}" ixy="0.0" ixz="0.0"
-                    iyy="${(1/12) * mass * (x*x+z*z)}" iyz="0.0"
-                    izz="${(1/12) * mass * (x*x+y*y)}" />
-        </inertial>
-    </xacro:macro>
-    <xacro:macro name="inertial_cylinder" params="mass length radius *origin">
-        <inertial>
-            <xacro:insert_block name="origin"/>
-            <mass value="${mass}" />
-            <inertia ixx="${(1/12) * mass * (3*radius*radius + length*length)}" ixy="0.0" ixz="0.0"
-                    iyy="${(1/12) * mass * (3*radius*radius + length*length)}" iyz="0.0"
-                    izz="${(1/2) * mass * (radius*radius)}" />
-        </inertial>
-    </xacro:macro>
-    <!-- <link name="world"></link> -->
-    <!-- <joint name="base_joint" type="fixed">
-        <origin xyz="1.5 1.0 0" rpy="0 0 0"/>
-        <parent link="world"/>
-        <child link="base_link"/>
-    </joint>
-    <link name="base_link">
-        <visual>
-            <origin xyz="0 0 0.05" rpy="0 0 0"/>
-            <geometry>
-                <box size="2.5 1.5 0.1" />
-            </geometry>
-            <material name="green">
-                <color rgba="0.2 1 0.2 1"/>
-            </material>
-        </visual>
-        <collision>
-            <origin xyz="0 0 0.05" rpy="0 0 0"/>
-            <geometry>
-                <box size="2.5 1.5 0.1" />
-            </geometry>
-        </collision>
-        <inertial>
-            <origin xyz="0 0 0.05" rpy="0 0 0"/>
-            <mass value="12" />
-            <inertia ixx="2.26" ixy="0.0" ixz="0.0" iyy="6.26" iyz="0.0" izz="8.5" />
-        </inertial>
-    </link>
-    <joint name="slider_joint_x" type="prismatic">
-        <origin xyz="-1.25 0 0.1" rpy="0 0 0"/>
-        <parent link="base_link"/>
-        <child link="slider_link"/>
-        <axis xyz="1 0 0"/>
-        <limit lower="-5" upper="5" velocity="100" effort="100"/>
-    </joint> -->
-    <!-- <link name="world"></link> -->
-    <!-- <joint name="world_joint" type="fixed">
-        <origin xyz="0 0 0" rpy="0 0 0"/>
-        <parent link="world"/>
-        <child link="slider_link"/>
-    </joint> -->
-    <link name="base_link">
-    </link>
-    <joint name="base_to_slider_joint" type="fixed">
-        <origin xyz="0 0 0" rpy="0 0 0"/>
-        <parent link="base_link"/>
-        <child link="slider_link"/>
-    </joint>
-    <link name="slider_link">
-        <visual>
-            <origin xyz="0 0 0.075" rpy="0 0 0"/>
-            <geometry>
-                <box size="0.5 0.25 0.15" />
-            </geometry>
-            <material name="blue" />
-        </visual>
-        <collision>
-            <origin xyz="0 0 0.075" rpy="0 0 0"/>
-            <geometry>
-                <box size="0.5 0.25 0.15" />
-            </geometry>
-        </collision>
-        <xacro:inertial_box mass="0.5" x="0.5" y="0.25" z="0.15">
-            <origin xyz="0 0 0" rpy="0 0 0"/>
-        </xacro:inertial_box>
-    </link>
-    <gazebo>
-        <!-- <plugin name="gazebo_ros_joint_state_publisher"
-            filename="libgazebo_ros_joint_state_publisher.so">
-            <update_rate>20</update_rate>
-            <joint_name>slider_joint_x</joint_name>
-            <joint_name>base_joint</joint_name>
-        </plugin> -->
-        <!-- model plugins must be inside the model tags to work -->
-        <!-- <plugin name="gazebo_ros_6dof_joint_state_publisher"
-            filename="libgazebo_ros_6dof_joint_state_publisher.so">
-        </plugin> -->
-        <plugin name="gazebo_ros_link_pose_publisher"
-            filename="libgazebo_ros_link_pose_publisher.so">
-        </plugin>
-    </gazebo>
-    <!-- camera -->
-    <gazebo reference="slider_link">
-        <sensor type="camera" name="camera1">
-            <update_rate>30.0</update_rate>
-            <visualize>true</visualize>
-            <camera name="head">
-                <horizontal_fov>1.3962634</horizontal_fov>
-                <image>
-                    <width>800</width>
-                    <height>800</height>
-                    <format>R8G8B8</format>
-                </image>
-                <clip>
-                    <near>0.02</near>
-                    <far>300</far>
-                </clip>
-                <noise>
-                    <type>gaussian</type>
-                    <mean>0.0</mean>
-                    <stddev>0.007</stddev>
-                </noise>
-            </camera>
-            <plugin name="camera_controller" filename="libgazebo_ros_camera.so">
-                <alwaysOn>true</alwaysOn>
-                <updateRate>0.0</updateRate>
-                <cameraName>vslam/camera1</cameraName>
-                <imageTopicName>image_raw</imageTopicName>
-                <cameraInfoTopicName>camera_info</cameraInfoTopicName>
-                <frameName>camera_link</frameName>
-                <hackBaseline>0.07</hackBaseline>
-                <distortionK1>0.0</distortionK1>
-                <distortionK2>0.0</distortionK2>
-                <distortionK3>0.0</distortionK3>
-                <distortionT1>0.0</distortionT1>
-                <distortionT2>0.0</distortionT2>
-            </plugin>
-        </sensor>
-    </gazebo>
-</robot>
+/workspace/vslam_dev_ws/src/camera_gazebo/description/bu.xacro

File: vslam_dev_ws/install/camera_gazebo/share/camera_gazebo/description/camera.urdf.xacro (robot description, xacro)
@@ -1,4 +1 @@
-<?xml version="1.0"?>
-<robot xmlns:xacro="http://www.ros.org/wiki/xacro" name="cart_robot">
-    <xacro:include filename="camera_core.xacro"/>
-</robot>
+/workspace/vslam_dev_ws/src/camera_gazebo/description/camera.urdf.xacro

File: vslam_dev_ws/install/camera_gazebo/share/camera_gazebo/description/camera_core.xacro (robot description, xacro)
@@ -1,106 +1 @@
-<?xml version="1.0"?>
-<robot xmlns:xacro="http://www.ros.org/wiki/xacro" name="camera_robot">
-    <xacro:property name="camera_link" value="0.05" /> <!-- Size of square 'camera' box -->
-    <gazebo reference="camera_stand_link">
-        <material>Gazebo/Green</material>
-        <!-- <gravity>0.0</gravity> -->
-    </gazebo>
-    <!-- This first link called "world" is empty -->
-    <link name="world"/>
-    <!-- A simple fixed joint from our empty world link, to our base. -->
-    <!-- The base origin is offset from the world origin. -->
-    <joint name="world_to_stand" type="fixed">
-        <origin xyz="0 0 0" rpy="0 0 0"/>
-        <parent link="world"/>
-        <child link="camera_stand_link"/>
-    </joint>
-    <!-- <link name="dummy">
-    </link>
-    <joint name="dummy_to_camera_link" type="continuous">
-        <origin xyz="0 0 0" rpy="0 0 0"/>
-        <pose>0 0 1 0 0 0</pose>
-        <parent link="dummy"/>
-        <child link="camera_link"/>
-        <axis>
-            <xyz>0 0 1</xyz>
-        </axis>
-    </joint>   -->
-    <!-- Camera -->
-    <link name="camera_stand_link">
-        <collision>
-            <origin xyz="0 0 0" rpy="0 0 0"/>
-            <geometry>
-                <box size="${camera_link} ${camera_link} ${camera_link}"/>
-            </geometry>
-        </collision>
-        <visual>
-            <origin xyz="0 0 0" rpy="0 0 0"/>
-            <geometry>
-                <box size="${camera_link} ${camera_link} ${camera_link}"/>
-            </geometry>
-            <material name="green">
-                <color rgba="0.2 1 0.2 1"/>
-            </material>
-        </visual>
-        <inertial>
-            <mass value="1e-5" />
-            <origin xyz="0 0 0" rpy="0 0 0"/>
-            <inertia ixx="1e-6" ixy="0" ixz="0" iyy="1e-6" iyz="0" izz="1e-6" />
-        </inertial>
-    </link>
-    <joint name="stand_to_camera" type="prismatic">
-        <origin xyz="-1.25 0 0.1" rpy="0 0 0"/>
-        <parent link="camera_stand_link"/>
-        <child link="camera_link"/>
-        <axis xyz="1 0 0"/>
-        <limit lower="0" upper="2" velocity="100" effort="100"/>
-    </joint>
-    <link name="camera_link">
-    </link>
-    <!-- camera -->
-    <gazebo reference="camera_link">
-        <sensor type="camera" name="camera1">
-            <update_rate>30.0</update_rate>
-            <visualize>true</visualize>
-            <camera name="head">
-                <horizontal_fov>1.3962634</horizontal_fov>
-                <image>
-                    <width>800</width>
-                    <height>800</height>
-                    <format>R8G8B8</format>
-                </image>
-                <clip>
-                    <near>0.02</near>
-                    <far>300</far>
-                </clip>
-                <noise>
-                    <type>gaussian</type>
-                    <mean>0.0</mean>
-                    <stddev>0.007</stddev>
-                </noise>
-            </camera>
-            <plugin name="camera_controller" filename="libgazebo_ros_camera.so">
-                <alwaysOn>true</alwaysOn>
-                <updateRate>0.0</updateRate>
-                <cameraName>vslam/camera1</cameraName>
-                <imageTopicName>image_raw</imageTopicName>
-                <cameraInfoTopicName>camera_info</cameraInfoTopicName>
-                <frameName>camera_link</frameName>
-                <hackBaseline>0.07</hackBaseline>
-                <distortionK1>0.0</distortionK1>
-                <distortionK2>0.0</distortionK2>
-                <distortionK3>0.0</distortionK3>
-                <distortionT1>0.0</distortionT1>
-                <distortionT2>0.0</distortionT2>
-            </plugin>
-        </sensor>
-    </gazebo>
-    <!-- rate to publish to /joint_states topic -->
-    <gazebo>
-        <plugin name="gazebo_ros_joint_state_publisher"
-            filename="libgazebo_ros_joint_state_publisher.so">
-            <update_rate>100</update_rate>
-            <joint_name>base_joint</joint_name>
-        </plugin>
-    </gazebo>
-</robot>
+/workspace/vslam_dev_ws/src/camera_gazebo/description/camera_core.xacro

File: vslam_dev_ws/src/camera_gazebo/description/bu.xacro (robot description, xacro)
@@ -112,14 +112,4 @@
     </link>
     <gazebo>
-        <!-- <plugin name="gazebo_ros_joint_state_publisher"
-            filename="libgazebo_ros_joint_state_publisher.so">
-            <update_rate>20</update_rate>
-            <joint_name>slider_joint_x</joint_name>
-            <joint_name>base_joint</joint_name>
-        </plugin> -->
-        <!-- model plugins must be inside the model tags to work -->
-        <!-- <plugin name="gazebo_ros_6dof_joint_state_publisher"
-            filename="libgazebo_ros_6dof_joint_state_publisher.so">
-        </plugin> -->
         <plugin name="gazebo_ros_link_pose_publisher"
             filename="libgazebo_ros_link_pose_publisher.so">

File: vslam_dev_ws/src/camera_gazebo/description/camera.urdf.xacro (robot description, xacro)
@@ -1,4 +1,5 @@
 <?xml version="1.0"?>
-<robot xmlns:xacro="http://www.ros.org/wiki/xacro" name="cart_robot">
+<robot xmlns:xacro="http://www.ros.org/wiki/xacro" name="camera_robot">
+    <!-- does not work for some reason, causes gazebo to crash, bu.xacro works though -->
     <xacro:include filename="camera_core.xacro"/>
 </robot>

File: vslam_dev_ws/src/camera_gazebo/description/camera_core.xacro (robot description, xacro)
@@ -1,4 +1,5 @@
 <?xml version="1.0"?>
 <robot xmlns:xacro="http://www.ros.org/wiki/xacro" name="camera_robot">
+    <!-- does not work for some reason, causes gazebo to crash, bu.xacro works though -->
     <xacro:property name="camera_link" value="0.05" /> <!-- Size of square 'camera' box -->
     <gazebo reference="camera_stand_link">
@@ -97,5 +98,5 @@
     </gazebo>
     <!-- rate to publish to /joint_states topic -->
-    <gazebo>
+    <!-- <gazebo>
         <plugin name="gazebo_ros_joint_state_publisher"
             filename="libgazebo_ros_joint_state_publisher.so">
@@ -103,4 +104,9 @@
             <joint_name>base_joint</joint_name>
         </plugin>
+    </gazebo> -->
+    <gazebo>
+        <plugin name="gazebo_ros_link_pose_publisher"
+            filename="libgazebo_ros_link_pose_publisher.so">
+        </plugin>
     </gazebo>
 </robot>
